Commit message: 1d

File: snek.urdf (robot description, URDF)
Before this commit: robot robot, 6 links, 5 joints
Links:
- added link Link6, mass 1; collision box size=0.8817935628017661 0.84182481376378 0.8446988747329754; visual box size=0.8817935628017661 0.84182481376378 0.8446988747329754
- added link Link7, mass 1; collision box size=0.2114898580502207 0.5591218111656817 0.7479942878340984; visual box size=0.2114898580502207 0.5591218111656817 0.7479942878340984
- added link Link8, mass 1; collision box size=0.6996725876772368 0.45157209322011127 0.9591977203554907; visual box size=0.6996725876772368 0.45157209322011127 0.9591977203554907
- added link Link9, mass 1; collision box size=0.15533837951338125 0.964754777883407 0.5288217946721038; visual box size=0.15533837951338125 0.964754777883407 0.5288217946721038
- link Link0: geometry collision box size=0.19354453015341144 0.594224816552752 0.1666603013283151; visual box size=0.19354453015341144 0.594224816552752 0.1666603013283151
- link Link1: geometry collision box size=0.2794639762198379 0.13604148972411723 0.36345459771779987; visual box size=0.2794639762198379 0.13604148972411723 0.36345459771779987
- link Link2: geometry collision box size=0.7509594877141564 0.5541820853154241 0.5113348962188801; visual box size=0.7509594877141564 0.5541820853154241 0.5113348962188801
- link Link3: geometry collision box size=0.9674896620274364 0.8292906094191805 0.12894829787615014; visual box size=0.9674896620274364 0.8292906094191805 0.12894829787615014
- link Link4: geometry collision box size=0.3151714440042339 0.3289174219059261 0.11530285839195697; visual box size=0.3151714440042339 0.3289174219059261 0.11530285839195697
- link Link5: geometry collision box size=0.9461654991090619 0.4711307461047618 0.6062358560336331; visual box size=0.9461654991090619 0.4711307461047618 0.6062358560336331
Joints:
- added joint Link5_Link6: type revolute, parent Link5, child Link6, origin xyz=0 0.4711307461047618 0 rpy=0 0 0, axis 0 1 0, limit lower=-3.14159 upper=3.14159 effort=0.0 velocity=0.0
- added joint Link6_Link7: type planar, parent Link6, child Link7, origin xyz=0 0.84182481376378 0 rpy=0 0 0, axis 0 0 1, limit lower=-3.14159 upper=3.14159 effort=0.0 velocity=0.0
- added joint Link7_Link8: type fixed, parent Link7, child Link8, origin xyz=0 0.5591218111656817 0 rpy=0 0 0, axis 0 1 0, limit lower=-3.14159 upper=3.14159 effort=0.0 velocity=0.0
- added joint Link8_Link9: type floating, parent Link8, child Link9, origin xyz=0 0.45157209322011127 0 rpy=0 0 0, axis 0 0 1, limit lower=-3.14159 upper=3.14159 effort=0.0 velocity=0.0
- joint Link0_Link1: origin xyz=0 0.34998405586638587 0 rpy=0 0 0 -> xyz=0 0.594224816552752 0 rpy=0 0 0; type revolute -> prismatic
- joint Link1_Link2: axis 1 0 0 -> 0 0 1; origin xyz=0 0.3620889325974541 0 rpy=0 0 0 -> xyz=0 0.13604148972411723 0 rpy=0 0 0
- joint Link2_Link3: origin xyz=0 0.38889594817578405 0 rpy=0 0 0 -> xyz=0 0.5541820853154241 0 rpy=0 0 0; type revolute -> prismatic
- joint Link3_Link4: origin xyz=0 0.23242101404924526 0 rpy=0 0 0 -> xyz=0 0.8292906094191805 0 rpy=0 0 0; type revolute -> floating
- joint Link4_Link5: axis 0 1 0 -> 0 0 1; origin xyz=0 0.24616252617298157 0 rpy=0 0 0 -> xyz=0 0.3289174219059261 0 rpy=0 0 0; type revolute -> prismatic

Commit message: snek

File: snek.urdf (robot description, URDF)
Before this commit: robot robot, 10 links, 9 joints
Links:
- added link Link10, mass 1; collision box size=0.5068788797207014 0.539835913886719 1; visual box size=0.5068788797207014 0.539835913886719 1
- added link Link11, mass 1; collision box size=0.19121438420139036 0.11449841346857725 1; visual box size=0.19121438420139036 0.11449841346857725 1
- link Link0: geometry collision box size=0.24076451749156136 0.06729542063096994 1; visual box size=0.24076451749156136 0.06729542063096994 1
- link Link1: geometry collision box size=0.0005934001627746488 0.8769609472025404 1; visual box size=0.0005934001627746488 0.8769609472025404 1
- link Link2: geometry collision box size=0.1220448929916299 0.008128040793792035 1; visual box size=0.1220448929916299 0.008128040793792035 1
- link Link3: geometry collision box size=0.9061355757792764 0.7402183253810287 1; visual box size=0.9061355757792764 0.7402183253810287 1
- link Link4: geometry collision box size=0.7521586923805633 0.381776352629725 1; visual box size=0.7521586923805633 0.381776352629725 1
- link Link5: geometry collision box size=0.14783289117398668 0.8520384532320464 1; visual box size=0.14783289117398668 0.8520384532320464 1
- link Link6: geometry collision box size=0.975174371755142 0.7539708706456818 1; visual box size=0.975174371755142 0.7539708706456818 1
- link Link7: geometry collision box size=0.6991246240202236 0.38817997961495143 1; visual box size=0.6991246240202236 0.38817997961495143 1
- link Link8: geometry collision box size=0.15631120483730387 0.8706713398766176 1; visual box size=0.15631120483730387 0.8706713398766176 1
- link Link9: geometry collision box size=0.5864242139763272 0.9782018965205593 1; visual box size=0.5864242139763272 0.9782018965205593 1
Joints:
- added joint Link10_Link11: type prismatic, parent Link10, child Link11, origin xyz=0 0.539835913886719 0 rpy=0 0 0, axis 1 0 1, limit lower=-3.14159 upper=3.14159 effort=0.0 velocity=0.0
- added joint Link9_Link10: type revolute, parent Link9, child Link10, origin xyz=0 0.9782018965205593 0 rpy=0 0 0, axis 1 0 1, limit lower=-3.14159 upper=3.14159 effort=0.0 velocity=0.0
- joint Link0_Link1: axis 0 0 1 -> 1 0 1; origin xyz=0 0.594224816552752 0 rpy=0 0 0 -> xyz=0 0.03364771031548497 0 rpy=0 0 0; type prismatic -> revolute
- joint Link1_Link2: axis 0 0 1 -> 1 0 1; origin xyz=0 0.13604148972411723 0 rpy=0 0 0 -> xyz=0 0.8769609472025404 0 rpy=0 0 0; type revolute -> prismatic
- joint Link2_Link3: axis 0 1 0 -> 1 0 1; origin xyz=0 0.5541820853154241 0 rpy=0 0 0 -> xyz=0 0.008128040793792035 0 rpy=0 0 0; type prismatic -> revolute
- joint Link3_Link4: axis 1 0 0 -> 1 0 1; origin xyz=0 0.8292906094191805 0 rpy=0 0 0 -> xyz=0 0.7402183253810287 0 rpy=0 0 0; type floating -> prismatic
- joint Link4_Link5: axis 0 0 1 -> 1 0 1; origin xyz=0 0.3289174219059261 0 rpy=0 0 0 -> xyz=0 0.381776352629725 0 rpy=0 0 0
- joint Link5_Link6: axis 0 1 0 -> 1 0 1; origin xyz=0 0.4711307461047618 0 rpy=0 0 0 -> xyz=0 0.8520384532320464 0 rpy=0 0 0; type revolute -> prismatic
- joint Link6_Link7: axis 0 0 1 -> 1 0 1; origin xyz=0 0.84182481376378 0 rpy=0 0 0 -> xyz=0 0.7539708706456818 0 rpy=0 0 0; type planar -> revolute
- joint Link7_Link8: axis 0 1 0 -> 1 0 1; origin xyz=0 0.5591218111656817 0 rpy=0 0 0 -> xyz=0 0.38817997961495143 0 rpy=0 0 0; type fixed -> prismatic
- joint Link8_Link9: axis 0 0 1 -> 1 0 1; origin xyz=0 0.45157209322011127 0 rpy=0 0 0 -> xyz=0 0.8706713398766176 0 rpy=0 0 0; type floating -> revolute

Commit message: tardigrade

File: snek.urdf (robot description, URDF)
Before this commit: robot robot, 12 links, 11 joints
Links:
- link Link0: geometry collision box size=0.5158782353088323 0.4305128902608041 1; visual box size=0.5158782353088323 0.4305128902608041 1
- link Link1: geometry collision box size=0.481913867953362 0.4782471249089336 1; visual box size=0.481913867953362 0.4782471249089336 1
- link Link10: geometry collision box size=0.19043200279090766 0.49377692285375074 1; visual box size=0.19043200279090766 0.49377692285375074 1
- link Link11: geometry collision box size=0.5625540535779137 0.7364967854569149 1; visual box size=0.5625540535779137 0.7364967854569149 1
- link Link2: geometry collision box size=0.9212807170717402 0.05184439792213125 1; visual box size=0.9212807170717402 0.05184439792213125 1
- link Link3: geometry collision box size=0.5916650531485189 0.7550028488145444 1; visual box size=0.5916650531485189 0.7550028488145444 1
- link Link4: geometry collision box size=0.026231059509629562 0.17682982601506403 1; visual box size=0.026231059509629562 0.17682982601506403 1
- link Link5: geometry collision box size=0.5685082416546136 0.9322616993515089 1; visual box size=0.5685082416546136 0.9322616993515089 1
- link Link6: geometry collision box size=0.0069034529954210555 0.3923831623663452 1; visual box size=0.0069034529954210555 0.3923831623663452 1
- link Link7: geometry collision box size=0.9249278603154096 0.5305895254090224 1; visual box size=0.9249278603154096 0.5305895254090224 1
- link Link8: geometry collision box size=0.8719935547050015 0.620662744685775 1; visual box size=0.8719935547050015 0.620662744685775 1
- link Link9: geometry collision box size=0.8222195422317016 0.6969351849047658 1; visual box size=0.8222195422317016 0.6969351849047658 1
Joints:
- joint Link0_Link1: origin xyz=0 0.03364771031548497 0 rpy=0 0 0 -> xyz=0 0.21525644513040204 0 rpy=0 0 0; type revolute -> fixed
- joint Link10_Link11: origin xyz=0 0.539835913886719 0 rpy=0 0 0 -> xyz=0 0.49377692285375074 0 rpy=0 0 0; type prismatic -> revolute
- joint Link1_Link2: origin xyz=0 0.8769609472025404 0 rpy=0 0 0 -> xyz=0 0.4782471249089336 0 rpy=0 0 0; type prismatic -> fixed
- joint Link2_Link3: origin xyz=0 0.008128040793792035 0 rpy=0 0 0 -> xyz=0 0.05184439792213125 0 rpy=0 0 0
- joint Link3_Link4: origin xyz=0 0.7402183253810287 0 rpy=0 0 0 -> xyz=0 0.7550028488145444 0 rpy=0 0 0; type prismatic -> fixed
- joint Link4_Link5: origin xyz=0 0.381776352629725 0 rpy=0 0 0 -> xyz=0 0.17682982601506403 0 rpy=0 0 0
- joint Link5_Link6: origin xyz=0 0.8520384532320464 0 rpy=0 0 0 -> xyz=0 0.9322616993515089 0 rpy=0 0 0; type prismatic -> revolute
- joint Link6_Link7: origin xyz=0 0.7539708706456818 0 rpy=0 0 0 -> xyz=0 0.3923831623663452 0 rpy=0 0 0; type revolute -> fixed
- joint Link7_Link8: origin xyz=0 0.38817997961495143 0 rpy=0 0 0 -> xyz=0 0.5305895254090224 0 rpy=0 0 0
- joint Link8_Link9: origin xyz=0 0.8706713398766176 0 rpy=0 0 0 -> xyz=0 0.620662744685775 0 rpy=0 0 0
- joint Link9_Link10: origin xyz=0 0.9782018965205593 0 rpy=0 0 0 -> xyz=0 0.6969351849047658 0 rpy=0 0 0
