Commit message: stasdf

File: tardigrade0.urdf (robot description, URDF)
Before this commit: robot robot, 27 links, 26 joints
Links:
- removed link Link1Left
- removed link Link1LeftFoot
- removed link Link1Right
- removed link Link1RightFoot
- added link Link6, mass 1; collision box size=1 1 1; visual box size=1 1 1
- added link Link6Left, mass 1; collision box size=1 0.16666666666666666 0.16666666666666666; visual box size=1 0.16666666666666666 0.16666666666666666
- added link Link6LeftFoot, mass 1; collision box size=0.16666666666666666 0.16666666666666666 1; visual box size=0.16666666666666666 0.16666666666666666 1
- added link Link6Right, mass 1; collision box size=1 0.16666666666666666 0.16666666666666666; visual box size=1 0.16666666666666666 0.16666666666666666
- added link Link6RightFoot, mass 1; collision box size=0.16666666666666666 0.16666666666666666 1; visual box size=0.16666666666666666 0.16666666666666666 1
Joints:
- removed joint Link1Left_Link1LeftFoot
- removed joint Link1Right_Link1RightFoot
- removed joint Link1_Link1Left
- removed joint Link1_Link1Right
- added joint Link5_Link6: type fixed, parent Link5, child Link6, origin xyz=0 1 0 rpy=0 0 0, axis 0 1 0, limit lower=-3.14159 upper=3.14159 effort=0.0 velocity=0.0
- added joint Link6Left_Link6LeftFoot: type fixed, parent Link6Left, child Link6LeftFoot, origin xyz=1 0 0.5 rpy=0 0 0, axis 1 0 1, limit lower=-3.14159 upper=3.14159 effort=0.0 velocity=0.0
- added joint Link6Right_Link6RightFoot: type fixed, parent Link6Right, child Link6RightFoot, origin xyz=1 0 0.5 rpy=0 0 0, axis 1 0 1, limit lower=-3.14159 upper=3.14159 effort=0.0 velocity=0.0
- added joint Link6_Link6Left: type revolute, parent Link6, child Link6Left, origin xyz=0 0 0 rpy=0 0 0, axis 0 1 1, limit lower=-3.14159 upper=3.14159 effort=0.0 velocity=0.0
- added joint Link6_Link6Right: type revolute, parent Link6, child Link6Right, origin xyz=0 0 0 rpy=0 0 0, axis 0 1 1, limit lower=-3.14159 upper=3.14159 effort=0.0 velocity=0.0

File: tardigrade1.urdf (robot description, URDF)
Before this commit: robot robot, 17 links, 16 joints
Links:
- removed link Link2Left
- removed link Link2LeftFoot
- removed link Link2Right
- removed link Link2RightFoot
- added link Link1Left, mass 1; collision box size=1 0.16666666666666666 0.16666666666666666; visual box size=1 0.16666666666666666 0.16666666666666666
- added link Link1LeftFoot, mass 1; collision box size=0.16666666666666666 0.16666666666666666 1; visual box size=0.16666666666666666 0.16666666666666666 1
- added link Link1Right, mass 1; collision box size=1 0.16666666666666666 0.16666666666666666; visual box size=1 0.16666666666666666 0.16666666666666666
- added link Link1RightFoot, mass 1; collision box size=0.16666666666666666 0.16666666666666666 1; visual box size=0.16666666666666666 0.16666666666666666 1
- added link Link4, mass 1; collision box size=1 1 1; visual box size=1 1 1
- added link Link4Left, mass 1; collision box size=1 0.16666666666666666 0.16666666666666666; visual box size=1 0.16666666666666666 0.16666666666666666
- added link Link4LeftFoot, mass 1; collision box size=0.16666666666666666 0.16666666666666666 1; visual box size=0.16666666666666666 0.16666666666666666 1
- added link Link4Right, mass 1; collision box size=1 0.16666666666666666 0.16666666666666666; visual box size=1 0.16666666666666666 0.16666666666666666
- added link Link4RightFoot, mass 1; collision box size=0.16666666666666666 0.16666666666666666 1; visual box size=0.16666666666666666 0.16666666666666666 1
Joints:
- removed joint Link2Left_Link2LeftFoot
- removed joint Link2Right_Link2RightFoot
- removed joint Link2_Link2Left
- removed joint Link2_Link2Right
- added joint Link1Left_Link1LeftFoot: type fixed, parent Link1Left, child Link1LeftFoot, origin xyz=1 0 0.5 rpy=0 0 0, axis 1 0 1, limit lower=-3.14159 upper=3.14159 effort=0.0 velocity=0.0
- added joint Link1Right_Link1RightFoot: type fixed, parent Link1Right, child Link1RightFoot, origin xyz=1 0 0.5 rpy=0 0 0, axis 1 0 1, limit lower=-3.14159 upper=3.14159 effort=0.0 velocity=0.0
- added joint Link1_Link1Left: type revolute, parent Link1, child Link1Left, origin xyz=0 0 0 rpy=0 0 0, axis 0 1 1, limit lower=-3.14159 upper=3.14159 effort=0.0 velocity=0.0
- added joint Link1_Link1Right: type revolute, parent Link1, child Link1Right, origin xyz=0 0 0 rpy=0 0 0, axis 0 1 1, limit lower=-3.14159 upper=3.14159 effort=0.0 velocity=0.0
- added joint Link3_Link4: type fixed, parent Link3, child Link4, origin xyz=0 1 0 rpy=0 0 0, axis 0 1 0, limit lower=-3.14159 upper=3.14159 effort=0.0 velocity=0.0
- added joint Link4Left_Link4LeftFoot: type fixed, parent Link4Left, child Link4LeftFoot, origin xyz=1 0 0.5 rpy=0 0 0, axis 1 0 1, limit lower=-3.14159 upper=3.14159 effort=0.0 velocity=0.0
- added joint Link4Right_Link4RightFoot: type fixed, parent Link4Right, child Link4RightFoot, origin xyz=1 0 0.5 rpy=0 0 0, axis 1 0 1, limit lower=-3.14159 upper=3.14159 effort=0.0 velocity=0.0
- added joint Link4_Link4Left: type revolute, parent Link4, child Link4Left, origin xyz=0 0 0 rpy=0 0 0, axis 0 1 1, limit lower=-3.14159 upper=3.14159 effort=0.0 velocity=0.0
- added joint Link4_Link4Right: type revolute, parent Link4, child Link4Right, origin xyz=0 0 0 rpy=0 0 0, axis 0 1 1, limit lower=-3.14159 upper=3.14159 effort=0.0 velocity=0.0
