Commit message: push

File: matchup.urdf (robot description, URDF)
Before this commit: robot robot, 45 links, 44 joints
Joints:
- joint ArmLeftArm0Left_ArmLeftArm1Left: axis 1 1 1 -> 1 1 0
- joint ArmLeftArm0Right_ArmLeftArm1Right: axis 1 1 1 -> 1 1 0
- joint ArmLeftArm1Left_ArmLeftArm2Left: axis 1 1 1 -> 1 1 0
- joint ArmLeftArm1Right_ArmLeftArm2Right: axis 1 1 1 -> 1 1 0
- joint ArmLeftArm2Left_ArmLeftArm3Left: axis 1 1 1 -> 1 1 0
- joint ArmLeftArm2Right_ArmLeftArm3Right: axis 1 1 1 -> 1 1 0
- joint ArmLeftArm3Left_ArmLeftArm4Left: axis 1 1 1 -> 1 1 0
- joint ArmLeftArm3Right_ArmLeftArm4Right: axis 1 1 1 -> 1 1 0
- joint ArmRightArm0Left_ArmRightArm1Left: axis 1 1 1 -> 1 1 0
- joint ArmRightArm0Right_ArmRightArm1Right: axis 1 1 1 -> 1 1 0
- joint ArmRightArm1Left_ArmRightArm2Left: axis 1 1 1 -> 1 1 0
- joint ArmRightArm1Right_ArmRightArm2Right: axis 1 1 1 -> 1 1 0
- joint ArmRightArm2Left_ArmRightArm3Left: axis 1 1 1 -> 1 1 0
- joint ArmRightArm2Right_ArmRightArm3Right: axis 1 1 1 -> 1 1 0
- joint ArmRightArm3Left_ArmRightArm4Left: axis 1 1 1 -> 1 1 0
- joint ArmRightArm3Right_ArmRightArm4Right: axis 1 1 1 -> 1 1 0
- joint RootLeft_SpineBaseLeft: axis 1 1 0 -> 1 0 0
- joint RootRight_SpineBaseRight: axis 1 1 0 -> 1 0 0
- joint Spine0Left_Spine1Left: axis 0 1 0 -> 1 1 0
- joint Spine0Right_Spine1Right: axis 0 1 0 -> 1 1 0
- joint Spine1Left_Spine2Left: axis 0 1 0 -> 1 1 0
- joint Spine1Right_Spine2Right: axis 0 1 0 -> 1 1 0
- joint Spine2Left_Spine3Left: axis 0 1 0 -> 1 1 0
- joint Spine2Right_Spine3Right: axis 0 1 0 -> 1 1 0
- joint Spine3Left_Spine4Left: axis 0 1 0 -> 1 1 0
- joint Spine3Right_Spine4Right: axis 0 1 0 -> 1 1 0
- joint Spine4Left_ArmLeftArm0Left: axis 1 1 1 -> 1 1 0
- joint Spine4Left_ArmRightArm0Left: axis 1 1 1 -> 1 1 0
- joint Spine4Right_ArmLeftArm0Right: axis 1 1 1 -> 1 1 0
- joint Spine4Right_ArmRightArm0Right: axis 1 1 1 -> 1 1 0
- joint SpineBaseLeft_Spine0Left: axis 0 1 0 -> 1 1 0; origin xyz=0 5 0.5 rpy=0 0 0 -> xyz=0 2.5 0.5 rpy=0 0 0
- joint SpineBaseRight_Spine0Right: axis 0 1 0 -> 1 1 0; origin xyz=0 -5 0.5 rpy=0 0 0 -> xyz=0 -2.5 0.5 rpy=0 0 0
